File: pcb/LoraHarvesterBox.kicad_sch (KiCad schematic)
At the start: 42 parts, among them J1 Conn_01x02_Pin, J2 Conn_01x02_Pin, J3 Conn_01x02_Pin, J4 Conn_01x04_Socket, J5 Conn_01x04_Socket, J6 Conn_01x04_Socket, J7 Conn_01x04_Socket, J8 Conn_01x06_Socket, SW1 SSSS811101, SW2 TS-1088-AR02016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

Commit message: pch, sch: use 0805 capacitor for FRAM and not 0402
Parts:
- C7: footprint Capacitor_SMD:C_0402_1005Metric_Pad0.74x0.62mm_HandSolder -> Capacitor_SMD:C_0805_2012Metric_Pad1.18x1.45mm_HandSolder
Changed lines of the file:
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@@
 			)
 		)
-		(property "Footprint" "Capacitor_SMD:C_0402_1005Metric_Pad0.74x0.62mm_HandSolder"
+		(property "Footprint" "Capacitor_SMD:C_0805_2012Metric_Pad1.18x1.45mm_HandSolder"
 			(at 61.9252 55.88 0)
 			(effects

Commit message: pcb, sch, doc: remove remaining 0401
Parts:
- C2, C3, C8: footprint Capacitor_SMD:C_0402_1005Metric_Pad0.74x0.62mm_HandSolder -> Capacitor_SMD:C_0603_1608Metric_Pad1.08x0.95mm_HandSolder
Changed lines of the file:
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@@
 			)
 		)
-		(property "Footprint" "Capacitor_SMD:C_0402_1005Metric_Pad0.74x0.62mm_HandSolder"
+		(property "Footprint" "Capacitor_SMD:C_0603_1608Metric_Pad1.08x0.95mm_HandSolder"
 			(at 50.4952 179.07 0)
 			(effects
@@
 			)
 		)
-		(property "Footprint" "Capacitor_SMD:C_0402_1005Metric_Pad0.74x0.62mm_HandSolder"
+		(property "Footprint" "Capacitor_SMD:C_0603_1608Metric_Pad1.08x0.95mm_HandSolder"
 			(at 130.5052 157.48 0)
 			(effects
@@
 			)
 		)
-		(property "Footprint" "Capacitor_SMD:C_0402_1005Metric_Pad0.74x0.62mm_HandSolder"
+		(property "Footprint" "Capacitor_SMD:C_0603_1608Metric_Pad1.08x0.95mm_HandSolder"
 			(at 155.9052 124.46 0)
 			(effects

Commit message: pcb, sch, doc: add buffer C for voltage dividers
Parts:
- added C10: 100nF, Capacitor_SMD:C_0603_1608Metric_Pad1.08x0.95mm_HandSolder, symbol Device:C
- added C9: 100nf, Capacitor_SMD:C_0603_1608Metric_Pad1.08x0.95mm_HandSolder, symbol Device:C
Connections:
- net ADC_BAT: now also C10.2
- net ADC_SOL: now also C9.2
- net GND: now also C10.1, C9.1
Changed lines of the file:
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@@
 	)
 	(junction
+		(at 41.91 102.87)
+		(diameter 0)
+		(color 0 0 0 0)
+	)
+	(junction
 		(at 33.02 58.42)
 		(diameter 0)
@@
 	)
 	(junction
+		(at 41.91 95.25)
+		(diameter 0)
+		(color 0 0 0 0)
+	)
+	(junction
 		(at 21.59 147.32)
 		(diameter 0)
@@
 	)
 	(junction
+		(at 24.13 102.87)
+		(diameter 0)
+		(color 0 0 0 0)
+	)
+	(junction
 		(at 215.9 198.12)
 		(diameter 0)
@@
 	(wire
 		(pts
+			(xy 20.32 102.87) (xy 24.13 102.87)
+		)
+		(stroke
+			(width 0)
+			(type default)
+		)
+	)
+	(wire
+		(pts
 			(xy 119.38 68.58) (xy 123.19 68.58)
 		)
@@
 	(wire
 		(pts
+			(xy 38.1 102.87) (xy 41.91 102.87)
+		)
+		(stroke
+			(width 0)
+			(type default)
+		)
+	)
+	(wire
+		(pts
 			(xy 36.83 55.88) (xy 33.02 55.88)
 		)
@@
 	(wire
 		(pts
+			(xy 20.32 95.25) (xy 20.32 92.71)
+		)
+		(stroke
+			(width 0)
+			(type default)
+		)
+	)
+	(wire
+		(pts
 			(xy 16.51 21.59) (xy 16.51 31.75)
 		)
@@
 	(wire
 		(pts
+			(xy 20.32 92.71) (xy 24.13 92.71)
+		)
+		(stroke
+			(width 0)
+			(type default)
+		)
+	)
+	(wire
+		(pts
 			(xy 215.9 198.12) (xy 215.9 200.66)
 		)
@@
 	(wire
 		(pts
+			(xy 38.1 95.25) (xy 41.91 95.25)
+		)
+		(stroke
+			(width 0)
+			(type default)
+		)
+	)
+	(wire
+		(pts
 			(xy 209.55 153.67) (xy 209.55 154.94)
 		)
@@
 	)
 	(symbol
+		(lib_id "Device:C")
+		(at 38.1 99.06 180)
+		(unit 1)
+		(exclude_from_sim no)
+		(in_bom yes)
+		(on_board yes)
+		(dnp no)
+		(property "Reference" "C10"
+			(at 36.83 101.6 0)
+			(effects
+				(font
+					(size 1.27 1.27)
+				)
+				(justify left)
+			)
+		)
+		(property "Value" "100nF"
+			(at 37.084 97.028 0)
+			(effects
+				(font
+					(size 1.27 1.27)
+				)
+				(justify left)
+			)
+		)
+		(property "Footprint" "Capacitor_SMD:C_0603_1608Metric_Pad1.08x0.95mm_HandSolder"
+			(at 37.1348 95.25 0)
+			(effects
+				(font
+					(size 1.27 1.27)
+				)
+				(hide yes)
+			)
+		)
+		(property "Datasheet" "~"
+			(at 38.1 99.06 0)
+			(effects
+				(font
+					(size 1.27 1.27)
+				)
+				(hide yes)
+			)
+		)
+		(property "Description" "Unpolarized capacitor"
+			(at 38.1 99.06 0)
+			(effects
+				(font
+					(size 1.27 1.27)
+				)
+				(hide yes)
+			)
+		)
+		(pin "1"
+		)
+		(pin "2"
+		)
+		(instances
+			(project "LoraHarvesterBox"
+				(path "/a6f37965-abbf-44d1-94f3-9a9b9eaa16a8"
+					(reference "C10")
+					(unit 1)
+				)
+			)
+		)
+	)
+	(symbol
 		(lib_id "power:GND")
 		(at 184.15 71.12 90)
@@
 					(unit 1)
 				)
+			)
+		)
+	)
+	(symbol
+		(lib_id "Device:C")
+		(at 20.32 99.06 180)
+		(unit 1)
+		(exclude_from_sim no)
+		(in_bom yes)
+		(on_board yes)
+		(dnp no)
+		(property "Reference" "C9"
+			(at 19.05 101.6 0)
+			(effects
+				(font
+					(size 1.27 1.27)
+				)
+				(justify left)
+			)
+		)
+		(property "Value" "100nf"
+			(at 19.304 97.028 0)
+			(effects
+				(font
+					(size 1.27 1.27)
+				)
+				(justify left)
+			)
+		)
+		(property "Footprint" "Capacitor_SMD:C_0603_1608Metric_Pad1.08x0.95mm_HandSolder"
+			(at 19.3548 95.25 0)
+			(effects
+				(font
+					(size 1.27 1.27)
+				)
+				(hide yes)
+			)
+		)
+		(property "Datasheet" "~"
+			(at 20.32 99.06 0)
+			(effects
+				(font
+					(size 1.27 1.27)
+				)
+				(hide yes)
+			)
+		)
+		(property "Description" "Unpolarized capacitor"
+			(at 20.32 99.06 0)
+			(effects
+				(font
+					(size 1.27 1.27)
+				)
+				(hide yes)
+			)
+		)
+		(pin "1"
+		)
+		(pin "2"
+		)
+		(instances
+			(project "LoraHarvesterBox"
+				(path "/a6f37965-abbf-44d1-94f3-9a9b9eaa16a8"
+					(reference "C9")
+					(unit 1)
+				)

Commit message: pcb, sch, doc: remove C as RAK31762 has 10uF+100nF already internally
Parts:
- removed C6: C, Capacitor_SMD:C_0805_2012Metric_Pad1.18x1.45mm_HandSolder, symbol Device:C
Changed lines of the file:
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@@
 	)
 	(junction
-		(at 201.93 55.88)
-		(diameter 0)
-		(color 0 0 0 0)
-	)
-	(junction
 		(at 41.91 102.87)
 		(diameter 0)
@@
 	(wire
 		(pts
-			(xy 173.99 55.88) (xy 201.93 55.88)
-		)
-		(stroke
-			(width 0)
-			(type default)
-		)
-	)
-	(wire
-		(pts
 			(xy 199.39 158.75) (xy 215.9 158.75)
 		)
@@
 	(wire
 		(pts
-			(xy 201.93 55.88) (xy 207.01 55.88)
+			(xy 173.99 55.88) (xy 182.88 55.88)
 		)
 		(stroke
@@
 	(wire
 		(pts
-			(xy 201.93 53.34) (xy 201.93 55.88)
-		)
-		(stroke
-			(width 0)
-			(type default)
-		)
-	)
-	(wire
-		(pts
 			(xy 119.38 71.12) (xy 123.19 71.12)
 		)
@@
 	(symbol
 		(lib_id "Device:C")
-		(at 201.93 49.53 0)
-		(unit 1)
-		(exclude_from_sim no)
-		(in_bom yes)
-		(on_board yes)
-		(dnp no)
-		(fields_autoplaced yes)
-		(property "Reference" "C6"
-			(at 205.74 48.2599 0)
-			(effects
-				(font
-					(size 1.27 1.27)
-				)
-				(justify left)
-			)
-		)
-		(property "Value" "C"
-			(at 205.74 50.7999 0)
-			(effects
-				(font
-					(size 1.27 1.27)
-				)
-				(justify left)
-			)
-		)
-		(property "Footprint" "Capacitor_SMD:C_0805_2012Metric_Pad1.18x1.45mm_HandSolder"
-			(at 202.8952 53.34 0)
-			(effects
-				(font
-					(size 1.27 1.27)
-				)
-				(hide yes)
-			)
-		)
-		(property "Datasheet" "~"
-			(at 201.93 49.53 0)
-			(effects
-				(font
-					(size 1.27 1.27)
-				)
-				(hide yes)
-			)
-		)
-		(property "Description" "Unpolarized capacitor"
-			(at 201.93 49.53 0)
-			(effects
-				(font
-					(size 1.27 1.27)
-				)
-				(hide yes)
-			)
-		)
-		(pin "2"
-		)
-		(pin "1"
-		)
-		(instances
-			(project ""
-				(path "/a6f37965-abbf-44d1-94f3-9a9b9eaa16a8"
-					(reference "C6")
-					(unit 1)
-				)
-			)
-		)
-	)
-	(symbol
-		(lib_id "Device:C")
 		(at 49.53 175.26 0)
 		(unit 1)
@@
 	(symbol
 		(lib_id "power:GND")
-		(at 201.93 45.72 180)
-		(unit 1)
-		(exclude_from_sim no)
-		(in_bom yes)
-		(on_board yes)
-		(dnp no)
-		(fields_autoplaced yes)
-		(property "Reference" "#PWR022"
-			(at 201.93 39.37 0)
-			(effects
-				(font
-					(size 1.27 1.27)
-				)
-				(hide yes)
-			)
-		)
-		(property "Value" "GND"
-			(at 201.93 40.64 0)
-			(effects
-				(font
-					(size 1.27 1.27)
-				)
-			)
-		)
-		(property "Footprint" ""
-			(at 201.93 45.72 0)
-			(effects
-				(font
-					(size 1.27 1.27)
-				)
-				(hide yes)
-			)
-		)
-		(property "Datasheet" ""
-			(at 201.93 45.72 0)
-			(effects
-				(font
-					(size 1.27 1.27)
-				)
-				(hide yes)
-			)
-		)
-		(property "Description" "Power symbol creates a global label with name \"GND\" , ground"
-			(at 201.93 45.72 0)
-			(effects
-				(font
-					(size 1.27 1.27)
-				)
-				(hide yes)
-			)
-		)
-		(pin "1"
-		)
-		(instances
-			(project "SolarMeshRepeater"
-				(path "/a6f37965-abbf-44d1-94f3-9a9b9eaa16a8"
-					(reference "#PWR022")
-					(unit 1)
-				)
-			)
-		)
-	)
-	(symbol
-		(lib_id "power:GND")
 		(at 40.64 146.05 0)
 		(unit 1)
@@
 	(symbol
 		(lib_id "power:+3V0")
-		(at 207.01 55.88 270)
+		(at 182.88 55.88 270)
 		(unit 1)
 		(exclude_from_sim no)
@@
 		(dnp no)
 		(property "Reference" "#PWR021"
-			(at 203.2 55.88 0)
+			(at 179.07 55.88 0)
 			(effects
 				(font
@@
 		)
 		(property "Value" "+3V0"
-			(at 210.82 55.8799 90)
+			(at 186.69 55.8799 90)
 			(effects
 				(font
@@
 		)
 		(property "Footprint" ""
-			(at 207.01 55.88 0)
+			(at 182.88 55.88 0)
 			(effects
 				(font
@@
 		)
 		(property "Datasheet" ""
-			(at 207.01 55.88 0)
+			(at 182.88 55.88 0)
 			(effects
 				(font
@@
 		)
 		(property "Description" "Power symbol creates a global label with name \"+3V0\""
-			(at 207.01 55.88 0)
+			(at 182.88 55.88 0)
 			(effects
 				(font

Commit message: pcb, sch, doc: make more pins available on the back
Parts:
- added J9: Conn_01x08_Socket, Connector_PinHeader_1.00mm:PinHeader_1x08_P1.00mm_Vertical_SMD_Pin1Left, symbol Connector:Conn_01x08_Socket
Connections:
- net +3V0: now also J9.7 (Pin_7)
- net GND: now also J9.8 (Pin_8)
- net at U2.20 (PA9): now also J9.1 (Pin_1)
- net at U2.25 (PA10/PIN_A3): now also J9.2 (Pin_2)
- net at U2.26 (PB2/PIN_A2): now also J9.3 (Pin_3)
- net at U2.27 (PB12): now also J9.4 (Pin_4)
- net at U2.29 (PA0): now also J9.5 (Pin_5)
- net at U2.30 (PB5): now also J9.6 (Pin_6)
- no-connect marks 8 -> 2

Commit message: sch, pcb, doc: remove FRAM to the top layer
Parts:
- C7: footprint Capacitor_SMD:C_0805_2012Metric_Pad1.18x1.45mm_HandSolder -> Capacitor_SMD:C_0603_1608Metric_Pad1.08x0.95mm_HandSolder
- D1: footprint LED_SMD:LED_0603_1608Metric -> LED_SMD:LED_0603_1608Metric_Pad1.05x0.95mm_HandSolder
- J7: footprint Connector_JST:JST_PH_B4B-PH-K_1x04_P2.00mm_Vertical -> Connector_JST:JST_ZH_B4B-ZR_1x04_P1.50mm_Vertical
Changed lines of the file:
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@@
 			)
 		)
-		(property "Footprint" "Capacitor_SMD:C_0805_2012Metric_Pad1.18x1.45mm_HandSolder"
+		(property "Footprint" "Capacitor_SMD:C_0603_1608Metric_Pad1.08x0.95mm_HandSolder"
 			(at 61.9252 55.88 0)
 			(effects
@@
 			)
 		)
-		(property "Footprint" "LED_SMD:LED_0603_1608Metric"
+		(property "Footprint" "LED_SMD:LED_0603_1608Metric_Pad1.05x0.95mm_HandSolder"
 			(at 245.11 68.58 0)
 			(effects
@@
 			)
 		)
-		(property "Footprint" "Connector_JST:JST_PH_B4B-PH-K_1x04_P2.00mm_Vertical"
+		(property "Footprint" "Connector_JST:JST_ZH_B4B-ZR_1x04_P1.50mm_Vertical"
 			(at 59.69 16.51 0)
 			(effects

Commit message: sch, pcb: clean up BOM
Parts:
- C3: value 0.01uF -> 10nF
- C7, C8: value C -> 100nF
- C9: value 100nf -> 100nF
Changed lines of the file:
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@@
 			)
 		)
-		(property "Value" "C"
+		(property "Value" "100nF"
 			(at 53.34 176.5299 0)
 			(effects
@@
 			)
 		)
-		(property "Value" "C"
+		(property "Value" "100nF"
 			(at 64.77 53.3399 0)
 			(effects
@@
 			)
 		)
-		(property "Value" "100nf"
+		(property "Value" "100nF"
 			(at 19.304 97.028 0)
 			(effects
@@
 			)
 		)
-		(property "Value" "0.01uF"
+		(property "Value" "10nF"
 			(at 155.448 122.936 0)
 			(effects

Commit message: pcb, doc, sch: add load switch. VBAT_OK (optionally) can switch on/off the RAK3172
Parts:
- added U4: TPS22917DBV, Package_TO_SOT_SMD:SOT-23-6, symbol Power_Management:TPS22917DBV
Connections:
- net +3V0: now also U4.1 (VIN); no longer U2.24 (VDD)
- net GND: now also U4.2 (GND)
- net VBAT_OK: now also U4.3 (ON)
- new net Vdd_Input: U2.24 (VDD), U4.6 (VOUT)
- no-connect marks 2 -> 4
Changed lines of the file:
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@@
 	)
 	(no_connect
+		(at 127 201.93)
+	)
+	(no_connect
 		(at 123.19 63.5)
 	)
 	(no_connect
+		(at 106.68 201.93)
+	)
+	(no_connect
 		(at 123.19 48.26)
 	)
@@
 	(wire
 		(pts
+			(xy 127 199.39) (xy 130.81 199.39)
+		)
+		(stroke
+			(width 0)
+			(type default)
+		)
+	)
+	(wire
+		(pts
 			(xy 49.53 179.07) (xy 49.53 182.88)
 		)
@@
 	(wire
 		(pts
+			(xy 104.14 196.85) (xy 104.14 199.39)
+		)
+		(stroke
+			(width 0)
+			(type default)
+		)
+	)
+	(wire
+		(pts
 			(xy 173.99 133.35) (xy 173.99 137.16)
 		)
@@
 	(wire
 		(pts
+			(xy 104.14 204.47) (xy 106.68 204.47)
+		)
+		(stroke
+			(width 0)
+			(type default)
+		)
+	)
+	(wire
+		(pts
 			(xy 173.99 50.8) (xy 199.39 50.8)
 		)
@@
 	(wire
 		(pts
+			(xy 116.84 209.55) (xy 116.84 212.09)
+		)
+		(stroke
+			(width 0)
+			(type default)
+		)
+	)
+	(wire
+		(pts
 			(xy 205.74 39.37) (xy 209.55 39.37)
 		)
@@
 	(wire
 		(pts
+			(xy 104.14 199.39) (xy 106.68 199.39)
+		)
+		(stroke
+			(width 0)
+			(type default)
+		)
+	)
+	(wire
+		(pts
 			(xy 154.94 114.3) (xy 154.94 116.84)
 		)
@@
 		)
 	)
+	(label "Vdd_Input"
+		(at 130.81 199.39 0)
+		(effects
+			(font
+				(size 1.27 1.27)
+			)
+			(justify left bottom)
+		)
+	)
 	(label "VSTOR"
 		(at 171.45 128.27 90)
@@
 		)
 	)
+	(label "VBAT_OK"
+		(at 104.14 204.47 180)
+		(effects
+			(font
+				(size 1.27 1.27)
+			)
+			(justify right bottom)
+		)
+	)
 	(label "+3V0"
 		(at 77.47 21.59 90)
@@
 		)
 	)
+	(label "Vdd_Input"
+		(at 182.88 55.88 0)
+		(effects
+			(font
+				(size 1.27 1.27)
+			)
+			(justify left bottom)
+		)
+	)
 	(label "BOOT"
 		(at 176.53 63.5 0)
@@
 	)
 	(symbol
+		(lib_id "Power_Management:TPS22917DBV")
+		(at 116.84 201.93 0)
+		(unit 1)
+		(exclude_from_sim no)
+		(in_bom yes)
+		(on_board yes)
+		(dnp no)
+		(fields_autoplaced yes)
+		(property "Reference" "U4"
+			(at 116.84 191.77 0)
+			(effects
+				(font
+					(size 1.27 1.27)
+				)
+			)
+		)
+		(property "Value" "TPS22917DBV"
+			(at 116.84 194.31 0)
+			(effects
+				(font
+					(size 1.27 1.27)
+				)
+			)
+		)
+		(property "Footprint" "Package_TO_SOT_SMD:SOT-23-6"
+			(at 116.84 189.23 0)
+			(effects
+				(font
+					(size 1.27 1.27)
+				)
+				(hide yes)
+			)
+		)
+		(property "Datasheet" "http://www.ti.com/lit/ds/symlink/tps22917.pdf"
+			(at 118.11 219.71 0)
+			(effects
+				(font
+					(size 1.27 1.27)
+				)
+				(hide yes)
+			)
+		)
+		(property "Description" "1V to 5.5V, 2A, 80mΩ Ultra-Low Leakage Load Switch, SOT23-6"
+			(at 116.84 201.93 0)
+			(effects
+				(font
+					(size 1.27 1.27)
+				)
+				(hide yes)
+			)
+		)
+		(pin "4"
+		)
+		(pin "6"
+		)
+		(pin "2"
+		)
+		(pin "1"
+		)
+		(pin "3"
+		)
+		(pin "5"
+		)
+		(instances
+			(project ""
+				(path "/a6f37965-abbf-44d1-94f3-9a9b9eaa16a8"
+					(reference "U4")
+					(unit 1)
+				)
+			)
+		)
+	)
+	(symbol
 		(lib_id "Device:R")
 		(at 228.6 199.39 0)
@@
 		(on_board yes)
 		(dnp no)
-		(fields_autoplaced yes)
 		(property "Reference" "#PWR010"
 			(at 215.9 137.16 0)
@@
 	)
 	(symbol
-		(lib_id "power:+3V0")
-		(at 182.88 55.88 270)
+		(lib_id "power:GND")
+		(at 116.84 212.09 0)
 		(unit 1)
 		(exclude_from_sim no)
@@
 		(on_board yes)
 		(dnp no)
+		(fields_autoplaced yes)
 		(property "Reference" "#PWR021"
-			(at 179.07 55.88 0)
+			(at 116.84 218.44 0)
 			(effects
 				(font
@@
 			)
 		)
-		(property "Value" "+3V0"
-			(at 186.69 55.8799 90)
+		(property "Value" "GND"
+			(at 116.84 217.17 0)
 			(effects
 				(font
 					(size 1.27 1.27)
 				)
-				(justify left)
 			)
 		)
 		(property "Footprint" ""
-			(at 182.88 55.88 0)
+			(at 116.84 212.09 0)
 			(effects
 				(font
@@
 		)
 		(property "Datasheet" ""
-			(at 182.88 55.88 0)
+			(at 116.84 212.09 0)
 			(effects
 				(font
@@
 			)
 		)
-		(property "Description" "Power symbol creates a global label with name \"+3V0\""
-			(at 182.88 55.88 0)
+		(property "Description" "Power symbol creates a global label with name \"GND\" , ground"
+			(at 116.84 212.09 0)
 			(effects
 				(font
@@
 		)
 		(instances
-			(project ""
+			(project "LoraHarvesterBox"
 				(path "/a6f37965-abbf-44d1-94f3-9a9b9eaa16a8"
 					(reference "#PWR021")
@@
 					(unit 1)
 				)
+			)
+		)
+	)
+	(symbol
+		(lib_id "power:+3V0")
+		(at 104.14 196.85 0)
+		(unit 1)
+		(exclude_from_sim no)
+		(in_bom yes)
+		(on_board yes)
+		(dnp no)
+		(fields_autoplaced yes)
+		(property "Reference" "#PWR041"
+			(at 104.14 200.66 0)
+			(effects
+				(font
+					(size 1.27 1.27)
+				)
+				(hide yes)
+			)
+		)
+		(property "Value" "+3V0"
+			(at 104.14 191.77 0)
+			(effects
+				(font
+					(size 1.27 1.27)
+				)
+			)
+		)
+		(property "Footprint" ""
+			(at 104.14 196.85 0)
+			(effects
+				(font
+					(size 1.27 1.27)
+				)
+				(hide yes)
+			)
+		)
+		(property "Datasheet" ""
+			(at 104.14 196.85 0)
+			(effects
+				(font
+					(size 1.27 1.27)
+				)
+				(hide yes)
+			)
+		)
+		(property "Description" "Power symbol creates a global label with name \"+3V0\""
+			(at 104.14 196.85 0)
+			(effects
+				(font
+					(size 1.27 1.27)
+				)
+				(hide yes)
+			)
+		)
+		(pin "1"
+		)
+		(instances
+			(project ""
+				(path "/a6f37965-abbf-44d1-94f3-9a9b9eaa16a8"
+					(reference "#PWR041")
+					(unit 1)
+				)
